File: rx_switch.brd (EAGLE design)
At the start: 100 x 80 mm, 9 parts, among them IC1 AT90S2313S

Commit message: PCB design
Parts:
- CAMERA: value CAMERA -> (none)
- IC1: value AT90S2313S -> (none)
- ISP: value ISP -> (none)
- RC_IN: value RC IN -> (none)
- moved C2 5.39 mm to (19.1, 16.5)
- renumbered SV1 to RC_IN, SV2 to CAMERA, SV3 to ISP
Connections:
- net N$7 renamed ISP
Routing:
- net VCC: track 0.00 -> 63.5 mm, vias 0 -> 1
- net GND: track 30.3 -> 60.9 mm, vias 0 -> 2
- net N$4: track 0.00 -> 26.0 mm
- net N$5: track 0.00 -> 24.7 mm
- net N$3: track 0.00 -> 21.5 mm
- net N$1: track 0.00 -> 19.1 mm
- net N$10: track 0.00 -> 16.4 mm, vias 0 -> 1
- net N$6: track 0.00 -> 9.58 mm, vias 0 -> 1
- net ISP: track 0.00 -> 8.31 mm
- net N$9: track 0.00 -> 7.52 mm, vias 0 -> 1
- net N$2: track 0.00 -> 5.77 mm
- net N$8: track 0.00 -> 3.51 mm, vias 0 -> 1
- net N$11: track 0.00 -> 3.51 mm, vias 0 -> 1
Other:
- board size 100 x 80 mm -> 34 x 19 mm
- board text added: "Janne Mäntyharju (c) 2013"
- board text added: "NXShutter"
- board text added: "V 2.0"

Commit message: PCB revision v.21
Parts:
- added ID: TPPAD1-13, testpad:P1-13
- added R3: 82K, rcl:R1206
- GREEN: value GREEN -> (none)
- R1: value 160 -> 150
- R2: value 130 -> 100
- RED: value RED -> (none)
- renumbered C2 to C1, LED1 to RED, LED2 to GREEN
Connections:
- new net N$7: ID.TP, R3.2
- net GND: now also R3.1
Routing:
- net GND: track 60.9 -> 72.6 mm
- net N$7: track 0.00 -> 2.94 mm
Other:
- board text added: "V 2.1"
- board text removed: "V 2.0"
Changed lines of the file:
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@@
 <?xml version="1.0" encoding="utf-8"?>
 <!DOCTYPE eagle SYSTEM "eagle.dtd">
-<eagle version="6.5.0">
+<eagle version="6.1">
 <drawing>
 <settings>
@@
 <setting verticaltext="up"/>
 </settings>
-<grid distance="0.05" unitdist="inch" unit="inch" style="lines" multiple="1" display="no" altdistance="0.025" altunitdist="inch" altunit="inch"/>
+<grid distance="0" unitdist="inch" unit="inch" style="lines" multiple="1" display="no" altdistance="0" altunitdist="inch" altunit="inch"/>
 <layers>
 <layer number="1" name="Top" color="4" fill="1" visible="yes" active="yes"/>
@@
 <wire x1="0" y1="19.04" x2="0" y2="0" width="0" layer="20"/>
 <text x="12.7" y="6.35" size="1.27" layer="26" rot="MR0">NXShutter</text>
-<text x="12.7" y="3.81" size="1.27" layer="26" rot="MR0">V 2.0</text>
+<text x="12.7" y="3.81" size="1.27" layer="26" rot="MR0">V 2.1</text>
 <text x="33.02" y="1.27" size="1.27" layer="26" rot="MR0">Janne Mäntyharju (c) 2013</text>
 </plain>
@@
 </class>
 </classes>
-<designrules name="default">
+<designrules>
 <description language="de">&lt;b&gt;EAGLE Design Rules&lt;/b&gt;
 &lt;p&gt;
@@
 <attribute name="OC_FARNELL" value="unknown" x="45.72" y="33.02" size="1.778" layer="27" rot="R90" display="off"/>
 </element>
-<element name="LED1" library="eagle-ltspice" package="LED_1206" value="RED" x="29.21" y="5.08" smashed="yes">
+<element name="RED" library="eagle-ltspice" package="LED_1206" value="" x="29.21" y="5.08" smashed="yes">
 <attribute name="SPICEMODEL" value="NONE" x="45.72" y="-27.94" size="1.778" layer="27" display="off"/>
 <attribute name="SPICETYPE" value="diode" x="45.72" y="-27.94" size="1.778" layer="27" display="off"/>
 <attribute name="SPICEPREFIX" value="D" x="45.72" y="-27.94" size="1.778" layer="27" display="off"/>
-<attribute name="VALUE" x="26.67" y="2.54" size="1.27" layer="27"/>
-</element>
-<element name="LED2" library="eagle-ltspice" package="LED_1206" value="GREEN" x="29.21" y="8.89" smashed="yes">
+<attribute name="NAME" x="27.564128125" y="2.682640625" size="1.27" layer="25"/>
+<attribute name="VALUE" x="27.94" y="2.54" size="1.27" layer="27"/>
+</element>
+<element name="GREEN" library="eagle-ltspice" package="LED_1206" value="" x="29.21" y="8.89" smashed="yes">
 <attribute name="SPICEMODEL" value="NONE" x="58.42" y="-16.51" size="1.778" layer="27" display="off"/>
 <attribute name="SPICETYPE" value="diode" x="58.42" y="-16.51" size="1.778" layer="27" display="off"/>
 <attribute name="SPICEPREFIX" value="D" x="58.42" y="-16.51" size="1.778" layer="27" display="off"/>
-<attribute name="VALUE" x="26.67" y="6.35" size="1.27" layer="27"/>
-</element>
-<element name="R1" library="rcl" package="R1206" value="160" x="22.86" y="5.08" smashed="yes" rot="MR180">
+<attribute name="NAME" x="26.0606375" y="6.586675" size="1.27" layer="25"/>
+<attribute name="VALUE" x="27.94" y="6.35" size="1.27" layer="27"/>
+</element>
+<element name="R1" library="rcl" package="R1206" value="150" x="22.86" y="5.08" smashed="yes" rot="MR180">
 <attribute name="NAME" x="21.59" y="3.81" size="1.27" layer="26" rot="MR180"/>
 <attribute name="VALUE" x="17.78" y="3.81" size="1.27" layer="28" rot="MR180"/>
 </element>
-<element name="R2" library="rcl" package="R1206" value="130" x="22.86" y="8.89" smashed="yes" rot="MR180">
+<element name="R2" library="rcl" package="R1206" value="100" x="22.86" y="8.89" smashed="yes" rot="MR180">
 <attribute name="NAME" x="24.13" y="11.43" size="1.27" layer="26" rot="MR180"/>
 <attribute name="VALUE" x="20.32" y="11.43" size="1.27" layer="28" rot="MR180"/>
 </element>
-<element name="C2" library="rcl" package="C0805" value="100nF" x="19.05" y="16.51" rot="MR0"/>
+<element name="C1" library="rcl" package="C0805" value="100nF" x="19.05" y="16.51" rot="MR0"/>
+<element name="R3" library="rcl" package="R1206" value="82K" x="6.7556875" y="5.094240625" smashed="yes" rot="R180">
+<attribute name="NAME" x="11.45203125" y="4.720996875" size="1.27" layer="25" rot="R180"/>
+<attribute name="VALUE" x="8.0256875" y="7.634240625" size="1.27" layer="27" rot="R180"/>
+</element>
+<element name="ID" library="testpad" package="P1-13" value="TPPAD1-13" x="2.400478125" y="5.08529375" smashed="yes">
+<attribute name="TP_SIGNAL_NAME" value="" x="1.130478125" y="2.54529375" size="1" layer="37"/>
+<attribute name="NAME" x="1.557446875" y="2.30090625" size="1.27" layer="25" ratio="10"/>
+<attribute name="VALUE" x="2.259528125" y="5.461434375" size="0.0254" layer="27"/>
+</element>
 </elements>
 <signals>
@@
 <contactref element="RC_IN" pad="1"/>
 <contactref element="IC1" pad="10"/>
-<contactref element="C2" pad="2"/>
+<contactref element="C1" pad="2"/>
 <contactref element="CAMERA" pad="1"/>
 <contactref element="ISP" pad="6"/>
-<contactref element="LED1" pad="C"/>
-<contactref element="LED2" pad="C"/>
+<contactref element="RED" pad="C"/>
+<contactref element="GREEN" pad="C"/>
 <wire x1="3.81" y1="13.97" x2="10.16" y2="13.97" width="0.6096" layer="1"/>
 <wire x1="30.632" y1="5.08" x2="30.632" y2="8.89" width="0.6096" layer="1"/>
@@
 <wire x1="27.94" y1="17.78" x2="18.1" y2="17.78" width="0.6096" layer="16"/>
 <wire x1="18.1" y1="17.78" x2="18.1" y2="16.51" width="0.6096" layer="16"/>
+<contactref element="R3" pad="1"/>
+<wire x1="8.1776875" y1="5.094240625" x2="7.75236875" y2="5.094240625" width="0.8128" layer="1"/>
+<wire x1="7.75236875" y1="5.094240625" x2="7.75236875" y2="13.870140625" width="0.8128" layer="1"/>
+<wire x1="7.75236875" y1="13.870140625" x2="10.16" y2="13.870140625" width="0.6096" layer="1"/>
+<wire x1="10.16" y1="13.870140625" x2="10.16" y2="13.97" width="0.6096" layer="1"/>
 </signal>
 <signal name="N$1">
@@
 <contactref element="RC_IN" pad="2"/>
 <contactref element="IC1" pad="20"/>
-<contactref element="C2" pad="1"/>
+<contactref element="C1" pad="1"/>
 <wire x1="3.81" y1="11.43" x2="6.35" y2="11.43" width="0.6096" layer="16"/>
 <wire x1="6.35" y1="11.43" x2="6.35" y2="1.27" width="0.6096" layer="16"/>
@@
 </signal>
 <signal name="N$8">
-<contactref element="LED1" pad="A"/>
+<contactref element="RED" pad="A"/>
 <contactref element="R1" pad="2"/>
 <wire x1="27.788" y1="5.08" x2="26.67" y2="5.08" width="0.6096" layer="1"/>
@@
 </signal>
 <signal name="N$11">
-<contactref element="LED2" pad="A"/>
+<contactref element="GREEN" pad="A"/>
 <contactref element="R2" pad="2"/>
 <wire x1="27.788" y1="8.89" x2="26.67" y2="8.89" width="0.6096" layer="1"/>
@@
 <wire x1="26.67" y1="8.89" x2="24.282" y2="8.89" width="0.6096" layer="16"/>
 </signal>
+<signal name="N$7">
+<contactref element="R3" pad="2"/>
+<contactref element="ID" pad="TP"/>
+<wire x1="5.3336875" y1="5.094240625" x2="2.400478125" y2="5.094240625" width="0.6096" layer="1"/>
+<wire x1="2.400478125" y1="5.094240625" x2="2.400478125" y2="5.08529375" width="0.6096" layer="1"/>
+</signal>
 </signals>

Commit message: Fixed NX500 / NX2000 support
Parts:
- R3: value 82K -> 68k
Changed lines of the file:
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@@
 </element>
 <element name="C1" library="rcl" package="C0805" value="100nF" x="19.05" y="16.51" rot="MR0"/>
-<element name="R3" library="rcl" package="R1206" value="82K" x="6.7556875" y="5.094240625" smashed="yes" rot="R180">
+<element name="R3" library="rcl" package="R1206" value="68k" x="6.7556875" y="5.094240625" smashed="yes" rot="R180">
 <attribute name="NAME" x="11.45203125" y="4.720996875" size="1.27" layer="25" rot="R180"/>
 <attribute name="VALUE" x="8.0256875" y="7.634240625" size="1.27" layer="27" rot="R180"/>
