File: rx_switch.sch (EAGLE design)
At the start: 4 parts, among them IC1 AT90S2313S

Commit message: Started creating pcb
Parts:
- removed C1: 100nF, rcl:C-EUC1812
- added C2: 100nF, rcl:C-EUC0805
- added LED1: RED, eagle-ltspice:LED_E
- added LED2: GREEN, eagle-ltspice:LED_E
- added R1: 160, rcl:R-EU_R1206
- added R2: 130, rcl:R-EU_R1206
- added SV3: ISP, con-lstb:MA03-2
Connections:
- new net N$1: IC1.RESET, SV3.5
- new net N$10: IC1.(TXD)PD1, R1.1
- new net N$11: LED2.A, R2.2
- new net N$6: IC1.(MISO)PB6, SV3.1
- new net N$7: IC1.(SCK)PB7, SV3.3
- new net N$8: LED1.A, R1.2
- new net N$9: IC1.(INT1)PD3, R2.1
- new net VCC: C2.1, IC1.VCC, SV1.2, SV3.2
- net GND: now also C2.2, LED1.C, LED2.C, SV3.6; no longer C1.1
- net N$2: now also IC1.(MOSI)PB5, SV3.4; no longer C1.2, IC1.VCC, SV1.2

Commit message: PCB design
Parts:
- CAMERA: value CAMERA -> (none)
- ISP: value ISP -> (none)
- RC_IN: value RC IN -> (none)
- renumbered SV1 to RC_IN, SV2 to CAMERA, SV3 to ISP
Connections:
- net N$7 renamed ISP
Changed lines of the file:
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@@
 </classes>
 <parts>
-<part name="SV1" library="con-lstb" deviceset="MA03-1" device="" value="RC IN"/>
-<part name="SV2" library="con-lstb" deviceset="MA03-1" device="" value="CAMERA"/>
+<part name="RC_IN" library="con-lstb" deviceset="MA03-1" device=""/>
+<part name="CAMERA" library="con-lstb" deviceset="MA03-1" device=""/>
 <part name="GND1" library="supply1" deviceset="GND" device=""/>
 <part name="GND2" library="supply1" deviceset="GND" device=""/>
-<part name="IC1" library="atmel" deviceset="AT90S2313" device="S"/>
-<part name="SV3" library="con-lstb" deviceset="MA03-2" device="" value="ISP"/>
+<part name="IC1" library="atmel" deviceset="AT90S2313" device="S" value=""/>
+<part name="ISP" library="con-lstb" deviceset="MA03-2" device=""/>
 <part name="GND3" library="supply1" deviceset="GND" device=""/>
 <part name="P+1" library="supply1" deviceset="VCC" device=""/>
@@
 </plain>
 <instances>
-<instance part="SV1" gate="G$1" x="35.56" y="22.86" rot="R90"/>
-<instance part="SV2" gate="G$1" x="78.74" y="68.58" rot="R180"/>
+<instance part="RC_IN" gate="G$1" x="35.56" y="22.86" rot="R90"/>
+<instance part="CAMERA" gate="G$1" x="78.74" y="68.58" rot="R180"/>
 <instance part="GND1" gate="1" x="43.18" y="33.02"/>
 <instance part="GND2" gate="1" x="76.2" y="81.28"/>
 <instance part="IC1" gate="G$1" x="33.02" y="60.96"/>
-<instance part="SV3" gate="1" x="33.02" y="96.52" rot="R180"/>
+<instance part="ISP" gate="1" x="33.02" y="96.52" rot="R180"/>
 <instance part="GND3" gate="1" x="43.18" y="91.44"/>
 <instance part="P+1" gate="VCC" x="5.08" y="68.58"/>
@@
 <net name="N$3" class="0">
 <segment>
-<pinref part="SV1" gate="G$1" pin="3"/>
+<pinref part="RC_IN" gate="G$1" pin="3"/>
 <wire x1="33.02" y1="30.48" x2="25.4" y2="30.48" width="0.1524" layer="91"/>
 <wire x1="25.4" y1="30.48" x2="25.4" y2="17.78" width="0.1524" layer="91"/>
@@
 <net name="N$4" class="0">
 <segment>
-<pinref part="SV2" gate="G$1" pin="2"/>
+<pinref part="CAMERA" gate="G$1" pin="2"/>
 <wire x1="71.12" y1="68.58" x2="50.8" y2="68.58" width="0.1524" layer="91"/>
 <pinref part="IC1" gate="G$1" pin="PB2"/>
@@
 <net name="N$5" class="0">
 <segment>
-<pinref part="SV2" gate="G$1" pin="3"/>
+<pinref part="CAMERA" gate="G$1" pin="3"/>
 <wire x1="71.12" y1="66.04" x2="50.8" y2="66.04" width="0.1524" layer="91"/>
 <pinref part="IC1" gate="G$1" pin="(AIN1)PB1"/>
@@
 <net name="GND" class="0">
 <segment>
-<pinref part="SV1" gate="G$1" pin="1"/>
+<pinref part="RC_IN" gate="G$1" pin="1"/>
 <wire x1="38.1" y1="30.48" x2="38.1" y2="35.56" width="0.1524" layer="91"/>
 <wire x1="38.1" y1="35.56" x2="15.24" y2="35.56" width="0.1524" layer="91"/>
@@
 </segment>
 <segment>
-<pinref part="SV2" gate="G$1" pin="1"/>
+<pinref part="CAMERA" gate="G$1" pin="1"/>
 <wire x1="71.12" y1="71.12" x2="71.12" y2="83.82" width="0.1524" layer="91"/>
 <pinref part="GND2" gate="1" pin="GND"/>
@@
 <segment>
 <pinref part="GND3" gate="1" pin="GND"/>
-<pinref part="SV3" gate="1" pin="6"/>
+<pinref part="ISP" gate="1" pin="6"/>
 <wire x1="43.18" y1="93.98" x2="40.64" y2="93.98" width="0.1524" layer="91"/>
 </segment>
@@
 <net name="N$1" class="0">
 <segment>
-<pinref part="SV3" gate="1" pin="5"/>
+<pinref part="ISP" gate="1" pin="5"/>
 <pinref part="IC1" gate="G$1" pin="RESET"/>
 <wire x1="25.4" y1="93.98" x2="15.24" y2="93.98" width="0.1524" layer="91"/>
@@
 <segment>
 <pinref part="P+2" gate="VCC" pin="VCC"/>
-<pinref part="SV3" gate="1" pin="2"/>
+<pinref part="ISP" gate="1" pin="2"/>
 <wire x1="45.72" y1="99.06" x2="40.64" y2="99.06" width="0.1524" layer="91"/>
 </segment>
 <segment>
-<pinref part="SV1" gate="G$1" pin="2"/>
+<pinref part="RC_IN" gate="G$1" pin="2"/>
 <wire x1="35.56" y1="30.48" x2="35.56" y2="33.02" width="0.1524" layer="91"/>
 <wire x1="35.56" y1="33.02" x2="5.08" y2="33.02" width="0.1524" layer="91"/>
@@
 <wire x1="50.8" y1="78.74" x2="55.88" y2="78.74" width="0.1524" layer="91"/>
 <wire x1="55.88" y1="78.74" x2="55.88" y2="101.6" width="0.1524" layer="91"/>
-<pinref part="SV3" gate="1" pin="1"/>
+<pinref part="ISP" gate="1" pin="1"/>
 <wire x1="55.88" y1="101.6" x2="25.4" y2="101.6" width="0.1524" layer="91"/>
 <wire x1="25.4" y1="101.6" x2="25.4" y2="99.06" width="0.1524" layer="91"/>
 </segment>
 </net>
-<net name="N$7" class="0">
+<net name="ISP" class="0">
 <segment>
-<pinref part="SV3" gate="1" pin="3"/>
+<pinref part="ISP" gate="1" pin="3"/>
 <wire x1="25.4" y1="96.52" x2="22.86" y2="96.52" width="0.1524" layer="91"/>
 <wire x1="22.86" y1="96.52" x2="22.86" y2="88.9" width="0.1524" layer="91"/>
@@
 <wire x1="50.8" y1="76.2" x2="53.34" y2="76.2" width="0.1524" layer="91"/>
 <wire x1="53.34" y1="76.2" x2="53.34" y2="96.52" width="0.1524" layer="91"/>
-<pinref part="SV3" gate="1" pin="4"/>
+<pinref part="ISP" gate="1" pin="4"/>
 <wire x1="53.34" y1="96.52" x2="40.64" y2="96.52" width="0.1524" layer="91"/>
 </segment>

Commit message: PCB revision v.21
Parts:
- added ID: TPPAD1-13, testpad:TPPAD1-13
- added R3: 82K, rcl:R-EU_R1206
- GREEN: value GREEN -> (none)
- R1: value 160 -> 150
- R2: value 130 -> 100
- RED: value RED -> (none)
- renumbered C2 to C1, LED1 to RED, LED2 to GREEN
Connections:
- new net N$7: ID.TP, R3.2
- net GND: now also R3.1
Changed lines of the file:
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@@
 <?xml version="1.0" encoding="utf-8"?>
 <!DOCTYPE eagle SYSTEM "eagle.dtd">
-<eagle version="6.5.0">
+<eagle version="6.1">
 <drawing>
 <settings>
@@
 <part name="P+1" library="supply1" deviceset="VCC" device=""/>
 <part name="P+2" library="supply1" deviceset="VCC" device=""/>
-<part name="LED1" library="eagle-ltspice" deviceset="LED_E" device="" value="RED"/>
-<part name="LED2" library="eagle-ltspice" deviceset="LED_E" device="" value="GREEN"/>
-<part name="R1" library="rcl" deviceset="R-EU_" device="R1206" value="160"/>
-<part name="R2" library="rcl" deviceset="R-EU_" device="R1206" value="130"/>
+<part name="RED" library="eagle-ltspice" deviceset="LED_E" device=""/>
+<part name="GREEN" library="eagle-ltspice" deviceset="LED_E" device=""/>
+<part name="R1" library="rcl" deviceset="R-EU_" device="R1206" value="150"/>
+<part name="R2" library="rcl" deviceset="R-EU_" device="R1206" value="100"/>
 <part name="GND4" library="supply1" deviceset="GND" device=""/>
-<part name="C2" library="rcl" deviceset="C-EU" device="C0805" value="100nF"/>
+<part name="C1" library="rcl" deviceset="C-EU" device="C0805" value="100nF"/>
+<part name="R3" library="rcl" deviceset="R-EU_" device="R1206" value="82K"/>
+<part name="ID" library="testpad" deviceset="TP" device="PAD1-13"/>
 </parts>
 <sheets>
@@
 <instance part="P+1" gate="VCC" x="5.08" y="68.58"/>
 <instance part="P+2" gate="VCC" x="48.26" y="99.06" rot="R270"/>
-<instance part="LED1" gate="G$1" x="71.12" y="45.72" rot="R90"/>
-<instance part="LED2" gate="G$1" x="78.74" y="50.8" rot="R90"/>
+<instance part="RED" gate="G$1" x="71.12" y="45.72" rot="R90"/>
+<instance part="GREEN" gate="G$1" x="78.74" y="50.8" rot="R90"/>
 <instance part="R1" gate="G$1" x="58.42" y="45.72"/>
 <instance part="R2" gate="G$1" x="63.5" y="50.8"/>
 <instance part="GND4" gate="1" x="93.98" y="43.18"/>
-<instance part="C2" gate="G$1" x="10.16" y="55.88" rot="R90"/>
+<instance part="C1" gate="G$1" x="10.16" y="55.88" rot="R90"/>
+<instance part="R3" gate="G$1" x="71.12" y="88.9" rot="R90"/>
+<instance part="ID" gate="G$1" x="71.12" y="101.6"/>
 </instances>
 <busses>
@@
 <pinref part="IC1" gate="G$1" pin="GND"/>
 <wire x1="15.24" y1="60.96" x2="15.24" y2="55.88" width="0.1524" layer="91"/>
-<pinref part="C2" gate="G$1" pin="2"/>
+<pinref part="C1" gate="G$1" pin="2"/>
 <wire x1="15.24" y1="55.88" x2="15.24" y2="35.56" width="0.1524" layer="91"/>
 <junction x="15.24" y="55.88"/>
@@
 <pinref part="GND2" gate="1" pin="GND"/>
 <wire x1="71.12" y1="83.82" x2="76.2" y2="83.82" width="0.1524" layer="91"/>
+<pinref part="R3" gate="G$1" pin="1"/>
+<junction x="71.12" y="83.82"/>
 </segment>
 <segment>
@@
 </segment>
 <segment>
-<pinref part="LED1" gate="G$1" pin="C"/>
+<pinref part="RED" gate="G$1" pin="C"/>
 <wire x1="76.2" y1="45.72" x2="88.9" y2="45.72" width="0.1524" layer="91"/>
 <wire x1="88.9" y1="45.72" x2="88.9" y2="50.8" width="0.1524" layer="91"/>
-<pinref part="LED2" gate="G$1" pin="C"/>
+<pinref part="GREEN" gate="G$1" pin="C"/>
 <wire x1="88.9" y1="50.8" x2="83.82" y2="50.8" width="0.1524" layer="91"/>
 <pinref part="GND4" gate="1" pin="GND"/>
@@
 <pinref part="P+1" gate="VCC" pin="VCC"/>
 <wire x1="5.08" y1="63.5" x2="5.08" y2="66.04" width="0.1524" layer="91"/>
-<pinref part="C2" gate="G$1" pin="1"/>
+<pinref part="C1" gate="G$1" pin="1"/>
 </segment>
 </net>
@@
 <net name="N$8" class="0">
 <segment>
-<pinref part="LED1" gate="G$1" pin="A"/>
+<pinref part="RED" gate="G$1" pin="A"/>
 <pinref part="R1" gate="G$1" pin="2"/>
 <wire x1="68.58" y1="45.72" x2="63.5" y2="45.72" width="0.1524" layer="91"/>
@@
 <net name="N$11" class="0">
 <segment>
-<pinref part="LED2" gate="G$1" pin="A"/>
+<pinref part="GREEN" gate="G$1" pin="A"/>
 <pinref part="R2" gate="G$1" pin="2"/>
 <wire x1="76.2" y1="50.8" x2="68.58" y2="50.8" width="0.1524" layer="91"/>
 </segment>
 </net>
+<net name="N$7" class="0">
+<segment>
+<pinref part="R3" gate="G$1" pin="2"/>
+<pinref part="ID" gate="G$1" pin="TP"/>
+<wire x1="71.12" y1="93.98" x2="71.12" y2="99.06" width="0.1524" layer="91"/>
+</segment>
+</net>

Commit message: Fixed NX500 / NX2000 support
Parts:
- R3: value 82K -> 68k
Other:
- note added: "black"
- note added: "green"
- note added: "white"
Changed lines of the file:
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@@
 <part name="GND4" library="supply1" deviceset="GND" device=""/>
 <part name="C1" library="rcl" deviceset="C-EU" device="C0805" value="100nF"/>
-<part name="R3" library="rcl" deviceset="R-EU_" device="R1206" value="82K"/>
+<part name="R3" library="rcl" deviceset="R-EU_" device="R1206" value="68k"/>
 <part name="ID" library="testpad" deviceset="TP" device="PAD1-13"/>
 </parts>
@@
 <sheet>
 <plain>
+<text x="73.66" y="76.2" size="1.778" layer="91">black</text>
+<text x="60.96" y="71.12" size="1.778" layer="91">green</text>
+<text x="60.96" y="63.5" size="1.778" layer="91">white</text>
 </plain>
 <instances>
